Commit message: add cover to robot

File: src/my_robot/urdf/my_robot.xacro (robot description, xacro)
@@ -55,4 +55,16 @@
       </geometry>
     </visual>
+    <collision name='cover_collision'>
+      <origin xyz="0 0 0.15" rpy=" 0 0 0"/>
+      <geometry>
+        <cylinder radius="0.25" length="0.01"/>
+      </geometry>
+    </collision>
+    <visual name='cover_visual'>
+      <origin xyz="0 0 0.15" rpy=" 0 0 0"/>
+      <geometry>
+        <cylinder radius="0.25" length="0.01"/>
+      </geometry>
+    </visual>
   </link>
   <link name='left_wheel'>

Commit message: add cover to robot

File: src/my_robot/urdf/my_robot.xacro (robot description, xacro)
@@ -193,11 +193,11 @@
   </joint>
   <gazebo reference="left_wheel">
-    <material>Gazebo/Green</material>
+    <material>Gazebo/Black</material>
   </gazebo>
   <gazebo reference="right_wheel">
-    <material>Gazebo/Green</material>
+    <material>Gazebo/Black</material>
   </gazebo>
   <gazebo reference="chassis">
-    <material>Gazebo/Blue</material>
+    <material>Gazebo/Black</material>
   </gazebo>
   <gazebo reference="camera">

Commit message: adding depthg camera and rtab slam

File: src/my_robot/urdf/my_robot.xacro (robot description, xacro)
@@ -140,16 +140,4 @@
       />
     </inertial>
-    <collision name='camera_collision'>
-      <origin xyz="0 0 0" rpy="0 0 0.0"/>
-      <geometry>
-        <box size="0.05 0.05 0.05"/>
-      </geometry>
-    </collision>
-    <visual name='camera_visual'>
-      <origin xyz="0 0 0" rpy="0 0 0.0"/>
-      <geometry>
-        <box size="0.05 0.05 0.05"/>
-      </geometry>
-    </visual>
   </link>
   <joint type="fixed" name="camera_joint">
@@ -157,5 +145,5 @@
     <child link="camera"/>
     <parent link="chassis"/>
-    <axis xyz="0 1 0" rpy="0 0 0"/>
+    <axis xyz="0 1 0" rpy="-1.5707 0 -1.5707"/>
     <limit effort="10000" velocity="1000"/>
     <dynamics damping="1.0" friction="1.0"/>
@@ -177,5 +165,5 @@
       </geometry>
     </collision>
-    <visual name='camera_visual'>
+    <visual name='hokuyo_visual'>
       <origin xyz="0 0 0" rpy="0 0 0.0"/>
       <geometry>
